File: TPDH-Walrus.sch (EAGLE design)
At the start: 45 parts, among them Q2 DMG3404, U1 MS5803-14BA, U2 SN65HVD33RHL, U4 MCP3421A3, U5 TPS79733, U6 MAX6070AAUT18, U7 TXS0102DQM

Commit message: Fixed thermistor divider, removed SDO
Changed thermistor voltage to VRef rather than 3v3, and removed connection to SDO pin.
Connections:
- net +3V3: no longer THERM.2
- net MISO: no longer U1.SDO
- net VREF: now also THERM.2

Commit message: power pad update; uniform board outline
Parts:
- PAD1, PAD10, PAD2, PAD3, PAD4, PAD5, PAD6, PAD7, PAD8, PAD9: device wirepad:1,6/0,8 -> wirepad:2,15/1,0

Commit message: Improved power layout, minor edits
Improved the overall layout of the power (3v3 and GND) as well as a few other minor edits. Changed orientation of I2C pins to match previous designs, also made pad on SN65HVD33 floating
Connections:
- net GND: no longer U2.EP
