File: TPDH-Walrus_v2_NoConn.brd (EAGLE design)
At the start: 16 x 40 mm, 35 parts, among them Q2 DMG3404, U1 MS5803-14BA, U2 SN65HVD72DSOIC, U4 MCP9808MSOP, U5 LP39883.3VDBV, U7 TXS0102DQM, U8 NS5A4684S

Commit message: Minor updates and cleanup, sent v2 NoConn to fab
Minor silkscreen and trace cleanup, sent v2 of through hole variant out to fab
Parts:
- removed C9: 0.1uF, bschulz_passives:C0402
- removed U8: NS5A4684S, bschulz:WQFN10
- added C7: 0.1uF, bschulz_passives:C0402
- added U6: (no value), bschulz:QFN20
- C2, C3: value 0.1uF -> 1uF; device bschulz_passives:C0402 -> bschulz:C0603
- C4, C5: value 1uF -> 0.1uF; device bschulz:C0603 -> bschulz_passives:C0402
- D1: value LEDBLUE0603 -> (none); device bschulz:LED_0603 -> bschulz:SOT23-3
- D2: value (none) -> LEDBLUE0603; device bschulz:SOT23-3 -> bschulz:LED_0603
- R1: value 1k -> 10k; device bschulz_passives:R0603 -> bschulz_passives:R0402
- R2: value 10k -> 100
- R4: value 10k -> 1k; device bschulz_passives:R0402 -> bschulz_passives:R0603
- R6: value 100 -> 10k
- U1: value MS5803-14BA -> MCP9808MSOP; device MS5803:MS5803 -> bschulz:MSOP_8
- U3: value (none) -> LP39883.3VDBV; device bschulz:QFN20 -> bschulz:DBV0005A
- U4: value MCP9808MSOP -> NS5A4684S; device bschulz:MSOP_8 -> bschulz:WQFN10
- U5: value LP39883.3VDBV -> TXS0102DQM; device bschulz:DBV0005A -> bschulz:DQM_R-PX2SON-N8
- U7: value TXS0102DQM -> MS580302BA; device bschulz:DQM_R-PX2SON-N8 -> bschulz:MS5803
- moved R5 29.9 mm to (0.88, 7.27)
- moved C6 26.1 mm to (4.29, 6.65), turned to 0 degrees
- moved R6 26.0 mm to (2.64, 37.1)
- moved R2 22.1 mm to (7.57, 11.5), turned to 270 degrees
- moved U4 21.1 mm to (6.05, 11.8)
- moved U7 18.7 mm to (8.00, 27.4), turned to 0 degrees
- moved C1 18.5 mm to (4.35, 32.8), turned to 90 degrees
- moved R1 15.7 mm to (11.8, 33.2), turned to 90 degrees
- moved R4 12.6 mm to (7.05, 18.2), turned to 180 degrees
- moved C5 12.0 mm to (5.28, 8.78), turned to 270 degrees
- moved C2 8.70 mm to (3.50, 15.3)
- moved D1 8.66 mm to (8.00, 8.10)
- moved D2 8.66 mm to (6.95, 16.7)
- moved U5 8.63 mm to (3.54, 9.28), turned to 180 degrees
- moved U3 7.17 mm to (3.95, 17.9), turned to 90 degrees
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- renumbered C10 to C8, Q2 to Q1, R8 to R7, U$12 to TP1
Connections:
- net !RESET: now also R6.1, U3.4, U6.12; no longer R5.1, U3.12, U5.4
- net +3V3: now also C4.1, C7.1, R1.2, R6.2, U1.8, U3.5, U5.1, U6.9, U7.6; no longer C6.1, C9.1, R2.2, R5.2, U1.5, U1.6, U3.9, U4.8, U7.1
- net A: now also R2.2, U4.10; no longer R6.2, U8.10
- net B: now also R2.1, U4.2; no longer R6.1, U8.2
- net GND: now also C7.2, D1.3, D2.CATHODE, U1.4, U1.5, U1.6, U1.7, U3.2, U5.4, U6.8, U6.EP, U7.2, U7.3; no longer C9.2, D1.CATHODE, D2.3, U1.2, U1.3, U3.8, U3.EP, U4.4, U4.5, U4.7, U5.2, U7.4, U8.6
- net MISO: now also U6.17; no longer U3.17
- net N$2: now also D2.ANODE, R4.1; no longer D1.ANODE, R1.1
- net OUTPUT_SEL: now also U4.4, U4.8, U6.1; no longer U3.1, U8.4, U8.8
- net PG: now also U6.13; no longer U3.13
- net REF_EN: now also U6.3; no longer U3.3
- net RX: now also U6.20; no longer U3.20
- net SCL: now also U5.2, U6.14; no longer U3.14, U7.2
- net SCL_HV: now also R5.1, U4.5, U5.7; no longer R4.1, U7.7, U8.5
- net SCL_OB: now also R1.1, U1.2, U6.4, U7.1; no longer R2.1, U1.1, U3.4, U4.2
- net SDA: now also U5.3, U6.18; no longer U3.18, U7.3
- net SDA_HV: now also U4.7, U5.6; no longer U7.6, U8.7
- net SDA_OB: now also U1.1, U6.5, U7.7; no longer U1.7, U3.5, U4.1
- net SIG1: now also D1.1, U4.9; no longer D2.1, U8.9
- net SIG2: now also D1.2, U4.3; no longer D2.2, U8.3
- net SN_DE: now also U6.15; no longer U3.15
- net SN_RE: now also U6.16; no longer U3.16
- net STAT_LED: now also R4.2, U6.2; no longer R1.2, U3.2
- net TEMP_ALERT: now also U1.3, U6.6; no longer U3.6, U4.3
- net TEST_PIN: now also U6.10; no longer U3.10
- net TX: now also U6.19; no longer U3.19
- net VIN+: now also C6.1, R5.2, U3.1, U3.3, U4.1, U5.8; no longer C4.1, R4.2, U5.1, U5.3, U7.8, U8.1
Routing:
- net +3V3: track 77.6 -> 75.9 mm
- net GND: track 89.8 -> 90.8 mm
Other:
- board text added: "Northern Widget"
- board text added: "Project-TPDH-Walrus v0.2.0 09-26-2019 Based on TP-Downhole by Schulz, Sandell, Wickert A. Wickert Northern Widget LLC and University of Minnesota"
- board text added: "Walrus v0.2"
- board text removed: "Project-TPDH-Walrus v0.2.0 07-15-2019 Based on TP-Downhole by Schulz, Sandell, Wickert A. Wickert Northern Widget LLC and University of Minnesota"
