File: TPDH-Walrus_v2_NoConn.sch (EAGLE design)
At the start: 35 parts, among them Q2 DMG3404, U1 MS5803-14BA, U2 SN65HVD72DSOIC, U4 MCP9808MSOP, U5 LP39883.3VDBV, U7 TXS0102DQM, U8 NS5A4684S

Commit message: Minor updates and cleanup, sent v2 NoConn to fab
Minor silkscreen and trace cleanup, sent v2 of through hole variant out to fab
Parts:
- removed C9: 0.1uF, bschulz_passives:C-EU0.1UFC0402
- removed U8: NS5A4684S, bschulz:NS5A4684S
- added C7: 0.1uF, bschulz_passives:C-EU0.1UFC0402
- added U6: (no value), bschulz:ATTINY1634QFN
- C2, C3: value 0.1uF -> 1uF; device bschulz_passives:C-EU0.1UFC0402 -> bschulz:C-EU1UFC0603
- C4, C5: value 1uF -> 0.1uF; device bschulz:C-EU1UFC0603 -> bschulz_passives:C-EU0.1UFC0402
- D1: value LEDBLUE0603 -> (none); device bschulz:LEDBLUE0603 -> bschulz:TVSSM712
- D2: value (none) -> LEDBLUE0603; device bschulz:TVSSM712 -> bschulz:LEDBLUE0603
- R1: value 1k -> 10k; device bschulz_passives:R-EU_1KR0603 -> bschulz_passives:R-EU_10KR0402
- R2: value 10k -> 100; device bschulz_passives:R-EU_10KR0402 -> bschulz_passives:R-EU_100R0402
- R4: value 10k -> 1k; device bschulz_passives:R-EU_10KR0402 -> bschulz_passives:R-EU_1KR0603
- R6: value 100 -> 10k; device bschulz_passives:R-EU_100R0402 -> bschulz_passives:R-EU_10KR0402
- U1: value MS5803-14BA -> MCP9808MSOP; device MS5803:MS5803-14BA -> bschulz:MCP9808MSOP; DIGIKEY 223-1625-5-ND -> (none); MF TE -> (none); MPN MS580305BA01-00 -> (none)
- U3: value (none) -> LP39883.3VDBV; device bschulz:ATTINY1634QFN -> bschulz:LP39883.3VDBV
- U4: value MCP9808MSOP -> NS5A4684S; device bschulz:MCP9808MSOP -> bschulz:NS5A4684S
- U5: value LP39883.3VDBV -> TXS0102DQM; device bschulz:LP39883.3VDBV -> bschulz:TXS0102DQM
- U7: value TXS0102DQM -> MS580302BA; device bschulz:TXS0102DQM -> bschulz:MS580302BA; DIGIKEY (none) -> 223-1625-5-ND; MF (none) -> TE; MPN (none) -> MS580305BA01-00
- renumbered C10 to C8, Q2 to Q1, R8 to R7, U$12 to TP1
Connections:
- net !RESET: now also R6.1, U3.PG, U6.PC3; no longer R5.1, U3.PC3, U5.PG
- net +3V3: now also C4.1, C7.1, R1.2, R6.2, U3.VOUT, U5.EN, U5.VA, U6.VCC, U7.PS, U7.VDD; no longer C6.1, C9.1, R2.2, R5.2, U1.PS, U3.VCC, U4.VDD, U5.VOUT, U7.EN, U7.VA
- net A: now also R2.2, U4.NO2; no longer R6.2, U8.NO2
- net B: now also R2.1, U4.NO1; no longer R6.1, U8.NO1
- net GND: now also C7.2, D1.COM, D2.CATHODE, U1.A0, U1.A1, U1.A2, U6.GND, U7.AD/CS; no longer C9.2, D1.CATHODE, D2.COM, U1.AD/CS, U4.A0, U4.A1, U4.A2, U8.GND
- net MISO: now also U6.PB2; no longer U3.PB2
- net N$2: now also D2.ANODE, R4.1; no longer D1.ANODE, R1.1
- net OUTPUT_SEL: now also U4.IN1, U4.IN2, U6.PA6; no longer U3.PA6, U8.IN1, U8.IN2
- net PG: now also U6.PC2; no longer U3.PC2
- net REF_EN: now also U6.PA4; no longer U3.PA4
- net RX: now also U6.PA7; no longer U3.PA7
- net SCL: now also U5.A1, U6.PC1; no longer U3.PC1, U7.A1
- net SCL_HV: now also R5.1, U4.NC1, U5.B1; no longer R4.1, U7.B1, U8.NC1
- net SCL_OB: now also R1.1, U1.SCL, U6.PA3, U7.SCL/SCLK; no longer R2.1, U1.SCL/SCLK, U3.PA3, U4.SCL
- net SDA: now also U5.A2, U6.PB1; no longer U3.PB1, U7.A2
- net SDA_HV: now also U4.NC2, U5.B2; no longer U7.B2, U8.NC2
- net SDA_OB: now also U1.SDA, U6.PA2, U7.SDA/SDI; no longer U1.SDA/SDI, U3.PA2, U4.SDA
- net SIG1: now also D1.D1, U4.COM2; no longer D2.D1, U8.COM2
- net SIG2: now also D1.D2, U4.COM1; no longer D2.D2, U8.COM1
- net SN_DE: now also U6.PC0; no longer U3.PC0
- net SN_RE: now also U6.PB3; no longer U3.PB3
- net STAT_LED: now also R4.2, U6.PA5; no longer R1.2, U3.PA5
- net TEMP_ALERT: now also U1.ALERT, U6.PA1; no longer U3.PA1, U4.ALERT
- net TEST_PIN: now also U6.PC5; no longer U3.PC5
- net TX: now also U6.PB0; no longer U3.PB0
- net VIN+: now also C6.1, R5.2, U3.EN, U3.VIN, U4.VCC, U5.VB; no longer C4.1, R4.2, U5.EN, U5.VIN, U7.VB, U8.VCC
Other:
- moved on the sheet: C1, C2, C3, C4, C5, C6, R1, R2, R4, R5, R6
