File: Hardware_HardMount/TPDH-Walrus_HardMount.brd (EAGLE design)
At the start: 12.7 x 42 mm, 30 parts, among them Q2 DMG3404, U1 MS5803-14BA, U2 SN65HVD72DSOIC, U4 MCP9808MSOP, U5 LP39883.3VDBV, U7 TXS0102DQM, U8 NS5A4684S

Commit message: Updated part numbers and BoM for HardMount variant
Updated part numbers in BoM to specifically indicate DNP where appropriate and to change MS5803 PN to 2BA model instead of 5BA model
Parts:
- LOGO1: device SparkFun-Aesthetics:OSHW-LOGO-M -> bschulz:OSHW-LOGO-M
- U1: value MS5803-14BA -> MS580302BA; device MS5803:MS5803 -> bschulz:MS5803
